File: corne-choc-wireless/pcb/corne-choc-wireless.kicad_pcb (KiCad board)
At the start: 2 copper layers, 275.5 x 105.6 mm, 118 parts, among them J2 Nice!View, J4 Nice!View, SW1 SW_PUSH, SW10 SW_PUSH, SW11 SW_PUSH, SW12 SW_PUSH, SW13 SW_PUSH, SW14 SW_PUSH, SW15 SW_PUSH, SW16 SW_PUSH, SW17 SW_PUSH, SW18 SW_PUSH, SW19 SW_PUSH, SW2 SW_PUSH, SW20 SW_PUSH, SW21 SW_PUSH, SW22 SW_PUSH, SW23 SW_PUSH, SW24 SW_PUSH, SW25 SW_PUSH, SW26 SW_PUSH, SW27 SW_PUSH, SW29 SW_PUSH, SW3 SW_PUSH, SW30 SW_PUSH, SW31 SW_PUSH, SW32 SW_PUSH, SW33 SW_PUSH, SW34 SW_PUSH, SW35 SW_PUSH, SW36 SW_PUSH, SW37 SW_PUSH, SW38 SW_PUSH, SW39 SW_PUSH, SW4 SW_PUSH, SW40 SW_PUSH, SW41 SW_PUSH, SW42 SW_PUSH, SW5 SW_PUSH, SW6 SW_PUSH, SW8 SW_PUSH, SW9 SW_PUSH, U1 Nice!Nano, U2 Nice!Nano

Commit message: Tweak roller pos
Parts:
- moved L_ENC1 0.22 mm to (21.7, 64.4)
- moved R_ENC1 0.09 mm to (279.3, 65.3)
Changed lines of the file:
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@@
   )
   (footprint "zzkeeb:RotaryEncoder_EVQWGD001" (layer "F.Cu")
-    (at 279.25 65.25 180)
+    (at 279.2725 65.3375 180)
     (property "Sheetfile" "corne-choc-wireless.kicad_sch")
     (property "Sheetname" "")
@@
   )
   (footprint "zzkeeb:RotaryEncoder_EVQWGD001" (layer "F.Cu")
-    (at 21.5175 64.2875)
-    (property "Sheetfile" "corne-choc-wireless.kicad_sch")
-    (property "Sheetname" "")
+    (at 21.71 64.39)
+    (property "Sheetfile" "corne-choc-wireless.kicad_sch")
+    (property "Sheetname" "")

Commit message: Filled zones
Routing:
- added copper zone on B.Cu, net (none)
- added copper zone on F.Cu, net (none)
Changed lines of the file:
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@@
   (segment (start 284.25 71.45) (end 283.027 72.673) (width 0.254) (layer "B.Cu") (net 84))
   (segment (start 284.25 71.45) (end 272.4875 59.6875) (width 0.254) (layer "B.Cu") (net 84))
+  (zone (net 0) (net_name "") (layers "F&B.Cu") (hatch edge 0.5)
+    (connect_pads (clearance 0.508))
+    (min_thickness 0.25) (filled_areas_thickness no)
+    (fill yes (thermal_gap 0.5) (thermal_bridge_width 0.5) (island_removal_mode 1) (island_area_min 10))
+    (polygon
+      (pts
+        (xy 0.02 0.18)
+        (xy 296.61 0.18)
+        (xy 296.99 209.98)
+        (xy -0.06 209.95)
+      )
+    )
+  )
   (group "" (id f4e27936-8ccc-4869-ab31-f3649459acab)
     (members

Commit message: Rotate right encoder
Parts:
- U1, U2: value Nice!Nano -> nice!nano
- moved D28 12.4 mm to (270.1, 64.9), turned to 90 degrees
- moved R_ENC1 1.58 mm to (277.9, 64.6), turned to 0 degrees
Routing:
- net GNDA: track 197.9 -> 179.0 mm, vias 2 -> 3
- net R_Enc_1: track 174.4 -> 159.1 mm
- net row1_r: track 120.9 -> 108.0 mm, vias 11 -> 9
- net R_ENC_B: track 114.5 -> 102.9 mm
- net R_ENC_A: track 113.5 -> 109.9 mm
- net col1_r: track 140.0 -> 137.0 mm
- net col2_r: track 120.9 -> 119.2 mm, vias 3 -> 1
- net R_Enc_2: track 6.17 -> 5.42 mm
Other:
- board text added: "Corne Cherry Wireless v1.0.0 PCB Designed by foostan & GSV-CargoCult"
- board text removed: "Corne Cherry v3.0.1 PCB Designed by foostan"

Commit message: Choc Done YAY
Parts:
- removed ? (x14): , 
- added G***: LOGO, LOGO, F.Cu at (222.2, 58.4)
- added G***: LOGO, kbd:corne-logo-horizontal, F.Cu at (269.7, 91.7)
- added G***: LOGO, kbd:corne-logo-horizontal, F.Cu at (31.7, 91.4)
- added G***: LOGO, LOGO, F.Cu at (82.7, 58.4)
- added G***: LOGO, kbd:corne-logo-horizontal, B.Cu at (60.3, 90.9)
- added G***: LOGO, kbd:corne-logo-horizontal, B.Cu at (240.9, 91.1)
- added Ref**: Val**, kbd:M2_HOLE_v2, F.Cu at (269.4, 55.4)
- added Ref**: Val**, kbd:M2_HOLE_v2, F.Cu at (193.4, 52.0)
- added Ref**: Val**, kbd:M2_HOLE_v2, B.Cu at (271.5, 64.3)
- added Ref**: Val**, kbd:M2_HOLE_v2, B.Cu at (171.1, 84.4)
- added Ref**: Val**, kbd:M2_HOLE_v2, B.Cu at (156.7, 93.0)
- added Ref**: Val**, kbd:M2_HOLE_v2, F.Cu at (144.4, 92.9)
- added Ref**: Val**, kbd:M2_HOLE_v2, F.Cu at (121.4, 99.3)
- added Ref**: Val**, kbd:M2_HOLE_v2, F.Cu at (74.9, 91.7)
- added Ref**: Val**, kbd:M2_HOLE_v2, F.Cu at (130.0, 84.4)
- added Ref**: Val**, kbd:M2_HOLE_v2, F.Cu at (29.6, 64.3)
- added Ref**: Val**, kbd:M2_HOLE_v2, F.Cu at (107.7, 51.9)
- added Ref**: Val**, kbd:M2_HOLE_v2, F.Cu at (31.7, 55.4)
- added Ref**: Val**, kbd:M2_HOLE_v2, F.Cu at (179.7, 99.3)
- SW1, SW10, SW11, SW12, SW13, SW14, SW15, SW16, SW17, SW18, SW19, SW2, SW20, SW22, SW23, SW24, SW25, SW26, SW27, SW29, SW3, SW30, SW31, SW32, SW33, SW34, SW35, SW36, SW37, SW38, SW39, SW4, SW40, SW41, SW5, SW6, SW8, SW9: footprint kbd:CherryMX_Hotswap -> Library:Hotswap_Choc_V1_MX_1.00u
- SW21, SW42: footprint kbd:CherryMX_Hotswap_1.5u -> ScottoKeebs_Hotswap:Hotswap_Choc_V1_1.50u
- U1, U2: value nice!nano -> Nice!Nano; footprint kbd:ProMicro_v3 -> ScottoKeebs_MCU:Nice_Nano_V2_Flipped
- moved D41 18.4 mm to (183.5, 98.5), turned to -75 degrees
- moved D19 18.1 mm to (80.0, 96.5), turned to -90 degrees
- moved D20 17.6 mm to (102.0, 97.0), turned to -105 degrees
- moved D6 16.7 mm to (108.2, 41.5), turned to -90 degrees
- moved D3 16.5 mm to (51.2, 40.5), turned to -90 degrees
- moved D34 16.5 mm to (270.2, 81.0), turned to -90 degrees
- moved D35 16.5 mm to (251.2, 81.0), turned to -90 degrees
- moved D39 16.5 mm to (175.2, 78.8), turned to -90 degrees
- moved D22 16.5 mm to (270.2, 43.2), turned to -90 degrees
- moved D23 16.5 mm to (251.2, 43.2), turned to -90 degrees
- moved D29 16.5 mm to (251.2, 62.2), turned to -90 degrees
- moved D14 16.5 mm to (32.5, 81.8), turned to -90 degrees
- moved D12 16.4 mm to (108.5, 60.2), turned to -90 degrees
- moved D18 16.4 mm to (108.5, 79.2), turned to -90 degrees
- moved D11 16.4 mm to (89.5, 58.0), turned to -90 degrees
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Routing:
- net row3_r: track 109.8 -> 73.5 mm, vias 0 -> 4
- net col5: track 96.2 -> 69.0 mm, vias 1 -> 0
- net row2_r: track 133.5 -> 115.5 mm, vias 6 -> 10
- net R_Enc_1: track 159.1 -> 174.9 mm, vias 1 -> 0
- net col3_r: track 124.6 -> 140.3 mm
- net row1_r: track 108.0 -> 94.9 mm, vias 9 -> 8
- net col1: track 137.0 -> 124.4 mm
- net row0: track 129.7 -> 142.1 mm, vias 10 -> 0
- net col1_r: track 137.0 -> 148.8 mm
- net col3: track 125.8 -> 114.0 mm
- net col2: track 117.7 -> 106.3 mm
- net L_Enc_2: track 15.5 -> 4.50 mm
- net row3: track 107.8 -> 117.2 mm, vias 0 -> 4
- net col2_r: track 119.2 -> 128.3 mm
- net row0_r: track 127.8 -> 118.9 mm, vias 11 -> 0
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