File: corne-cherry-wireless/pcb/corne-cherry-wireless.kicad_pcb (KiCad board)
At the start: 2 copper layers, 275.5 x 105.6 mm, 118 parts, among them J2 Nice!View, J4 Nice!View, SW1 SW_PUSH, SW10 SW_PUSH, SW11 SW_PUSH, SW12 SW_PUSH, SW13 SW_PUSH, SW14 SW_PUSH, SW15 SW_PUSH, SW16 SW_PUSH, SW17 SW_PUSH, SW18 SW_PUSH, SW19 SW_PUSH, SW2 SW_PUSH, SW20 SW_PUSH, SW21 SW_PUSH, SW22 SW_PUSH, SW23 SW_PUSH, SW24 SW_PUSH, SW25 SW_PUSH, SW26 SW_PUSH, SW27 SW_PUSH, SW29 SW_PUSH, SW3 SW_PUSH, SW30 SW_PUSH, SW31 SW_PUSH, SW32 SW_PUSH, SW33 SW_PUSH, SW34 SW_PUSH, SW35 SW_PUSH, SW36 SW_PUSH, SW37 SW_PUSH, SW38 SW_PUSH, SW39 SW_PUSH, SW4 SW_PUSH, SW40 SW_PUSH, SW41 SW_PUSH, SW42 SW_PUSH, SW5 SW_PUSH, SW6 SW_PUSH, SW8 SW_PUSH, SW9 SW_PUSH, U1 nice!nano, U2 nice!nano

Commit message: Replace rollers with switches
Parts:
- removed L_ENC1, R_ENC1: RollerEncoder_EVQWGD001, zzkeeb:RotaryEncoder_EVQWGD001
- added SW28: SW_PUSH, kbd:CherryMX_Hotswap, F.Cu at (278.9, 65.0)
- added SW7: SW_PUSH, kbd:CherryMX_Hotswap, F.Cu at (22.2, 65.0)
- U1, U2: value nice!nano -> Nice!Nano
- moved D28 16.4 mm to (286.5, 64.9)
Connections:
- net L_Enc_1 renamed col0
- net R_Enc_1 renamed col0_r
- D28 pad 2: R_Enc_2 -> Net-(D28-A)
- D7 pad 2: L_Enc_2 -> Net-(D7-A)
- U1 pad 13: L_ENC_B -> unconnected-(U1-D10-Pad13)
- U1 pad 14: L_ENC_A -> unconnected-(U1-D16-Pad14)
- U2 pad 11: R_ENC_B -> unconnected-(U2-D8-Pad11)
- U2 pad 12: R_ENC_A -> unconnected-(U2-D9-Pad12)
Routing:
- net GND: track 200.3 -> 69.8 mm
- net L_ENC_B: track 119.2 -> 0.00 mm
- net L_ENC_A: track 117.5 -> 0.00 mm
- net R_ENC_A: track 109.9 -> 0.00 mm
- net GNDA: track 179.0 -> 70.7 mm, vias 3 -> 2
- net R_ENC_B: track 102.9 -> 0.00 mm
- net row1_r: track 108.0 -> 127.9 mm, vias 9 -> 11
- net L_Enc_2: track 15.5 -> 0.00 mm
- net R_Enc_2: track 5.42 -> 0.00 mm
- net Net-(D7-A): track 0.00 -> 3.93 mm
- net Net-(D28-A): track 0.00 -> 3.75 mm
- net col0_r: track 159.1 -> 155.4 mm
- net col0: track 158.0 -> 155.1 mm, vias 0 -> 1
- net CS_r: track 33.6 -> 33.1 mm

Commit message: Replace promicro with nn
Parts:
- removed the ? at (74.9, 91.7)
- removed the ? at (144.4, 92.9)
- removed the ? at (31.7, 55.4)
- removed the ? at (31.7, 74.4)
- removed the ? at (130.0, 84.4)
- removed the ? at (121.4, 99.3)
- removed the ? at (107.7, 51.9)
- U1, U2: footprint kbd:ProMicro_v3 -> ScottoKeebs_MCU:Nice_Nano_V2_Flipped
- moved U1 0.60 mm to (136.9, 56.0)
- moved U2 0.60 mm to (164.2, 55.9)
Routing:
- net SCL: track 33.1 -> 35.2 mm
